Commit message: 增加rviz激光雷达点云输出，gazebo居家场景搭建

File: src/scout_description/urdf/chassis.xacro (robot description, xacro)
@@ -70,4 +70,44 @@
     <xacro:wheel_link prefix="front_right"/>
     <xacro:wheel_link prefix="rear_right"/>
+     <link name="laser_link">
+        <inertial>
+            <origin
+                xyz="0.0 0.0 0.0"
+                rpy="0 0 0" />
+            <mass
+                value="0.1" />
+            <inertia
+                ixx="0.0088463"
+                ixy="2.0356E-05"
+                ixz="-0.00047464"
+                iyy="0.0066478"
+                iyz="-6.9288E-06"
+                izz="0.01219" />
+        </inertial>
+        <visual>
+            <origin
+                    xyz="0.0 0.0 -0.047"
+                    rpy="0.0 0.0 0.0" />
+            <geometry>
+                    <mesh filename="package://scout_description/meshes/mid-360S.STL"/>
+            </geometry>
+            <material name = "white">
+            <color rgba="1 1 1 1" />
+            </material>
+        </visual>
+        <collision>
+            <origin
+                    xyz="0 0 -0.047"
+                    rpy="0 0 0" />
+          <geometry>
+                    <mesh filename="package://scout_description/meshes/mid-360S.STL"/>
+          </geometry>
+        </collision>
+    </link>
+    <joint name="laser_joint" type="fixed">
+        <origin xyz="0.21837 0 0.21508" rpy="0 0 0" />
+        <parent link="base_link" />
+        <child link="laser_link" />
+    </joint>
     <joint name="inertial_joint" type="fixed">
         <origin rpy="0 0 0" xyz="0 0 0"/>

Commit message: 增加piper机械臂与在gazebo当中的控制

File: src/scout_description/urdf/chassis.xacro (robot description, xacro)
@@ -105,4 +105,11 @@
         </collision>
     </link>
+    <link name="arm_link" />
+    <joint
+        name="arm_joint" type="fixed">
+        <origin xyz="0.06232 0 0.24623" rpy="0 0 0" />
+        <parent link="base_link" />
+        <child link="arm_link" />
+    </joint>
     <joint name="laser_joint" type="fixed">
         <origin xyz="0.21837 0 0.21508" rpy="0 0 0" />

File: src/scout_description/urdf/scout_mini.urdf.xacro (robot description, xacro)
@@ -4,4 +4,15 @@
     <xacro:include filename="common_properties.xacro" />
     <xacro:include filename="chassis.xacro" />
+    <xacro:include filename="/home/hanks/scout_ws/src/piper_description/urdf/my_robot.urdf.xacro" />
     <xacro:include filename="exp_in_sim.xacro" />
+    <joint
+        name="piper_base_joint"
+        type="fixed">
+        <parent
+            link="arm_link" />
+        <child
+            link="piper_base_link" />
+        <origin
+            xyz="0 0 0" rpy="0 0 0"/>
+    </joint>
 </robot>

Commit message: 加入fastlio2+nav2规划导航

File: src/scout_description/urdf/chassis.xacro (robot description, xacro)
@@ -70,5 +70,5 @@
     <xacro:wheel_link prefix="front_right"/>
     <xacro:wheel_link prefix="rear_right"/>
-     <link name="laser_link">
+     <link name="mid360_link">
         <inertial>
             <origin
@@ -106,4 +106,19 @@
     </link>
     <link name="arm_link" />
+    <link name="laser_link"/>
+    <!-- ==================== 新增：IMU 节点与物理连接 ==================== -->
+    <link name="imu_link">
+        <inertial>
+            <mass value="0.01"/>
+            <origin xyz="0 0 0" rpy="0 0 0"/>
+            <inertia ixx="0.00001" ixy="0" ixz="0" iyy="0.00001" iyz="0" izz="0.00001"/>
+        </inertial>
+    </link>
+    <!-- =================================================================== -->
+    <joint name="laser_link_alias_joint" type="fixed">
+        <parent link="mid360_link"/>
+        <child link="laser_link"/>
+        <origin xyz="0 0 0" rpy="0 0 0"/>
+    </joint>
     <joint
         name="arm_joint" type="fixed">
@@ -112,8 +127,13 @@
         <child link="arm_link" />
     </joint>
-    <joint name="laser_joint" type="fixed">
+    <joint name="mid360_joint" type="fixed">
         <origin xyz="0.21837 0 0.21508" rpy="0 0 0" />
         <parent link="base_link" />
-        <child link="laser_link" />
+        <child link="mid360_link" />
+    </joint>
+    <joint name="imu_joint" type="fixed">
+        <parent link="mid360_link"/>
+        <child link="imu_link"/>
+        <origin xyz="0.0 0.0 0.0" rpy="0 0 0"/>
     </joint>
     <joint name="inertial_joint" type="fixed">
@@ -151,3 +171,43 @@
         <axis rpy="0 0 0" xyz="0 0 -1"/>
     </joint>
+    <gazebo reference="mid360_joint">
+        <disableFixedJointLumping>true</disableFixedJointLumping>
+    </gazebo>
+    <!-- ==================== 新增：Gazebo IMU 仿真传感器配置 ==================== -->
+    <gazebo reference="imu_link">
+        <sensor name="imu_sensor" type="imu">
+            <always_on>true</always_on>
+            <update_rate>200</update_rate>
+            <topic>/livox/imu</topic>
+            <!-- 核心修改点：显式覆盖 frame_id 为 TF 树中存在的 link 名 -->
+            <gz_frame_id>imu_link</gz_frame_id>
+            <ignition_frame_id>imu_link</ignition_frame_id>
+            <plugin filename="gz-sim-imu-system" name="gz::sim::systems::Imu"/>
+        </sensor>
+    </gazebo>
+    <gazebo reference="front_left_wheel">
+        <mu1>5.0</mu1>
+        <mu2>5.0</mu2>
+    </gazebo>
+    <gazebo reference="rear_left_wheel">
+        <mu1>5.0</mu1>
+        <mu2>5.0</mu2>
+    </gazebo>
+    <gazebo reference="front_right_wheel">
+        <mu1>5.0</mu1>
+        <mu2>5.0</mu2>
+    </gazebo>
+    <gazebo reference="rear_right_wheel">
+        <mu1>5.0</mu1>
+        <mu2>5.0</mu2>
+    </gazebo>
+    <xacro:include
+        filename="$(find livox_mid360_gz_sim)/urdf/mid360_gz_plugin.xacro"/>
+    <xacro:livox_mid360_gz_plugin
+        link_name="mid360_link"
+        node_name="livox_mid360_gz_sim"
+        frame_id="laser_link"
+        topic="/livox/lidar"
+        points_topic="/livox/lidar/points"
+        update_rate="10.0"/>
 </robot>

File: src/scout_description/urdf/exp_in_sim.xacro (robot description, xacro)
@@ -5,4 +5,5 @@
             filename="gz-sim-diff-drive-system"
             name="gz::sim::systems::DiffDrive">
+            <wheels_per_side>2</wheels_per_side>
         <!-- 轮子关节名称 (需与你的 URDF 中的 joint 名一致) -->
             <left_joint>front_left_wheel</left_joint>
@@ -11,5 +12,5 @@
             <right_joint>rear_right_wheel</right_joint>
             <!-- 轮距与轮径 -->
-            <wheel_separation>0.4</wheel_separation>
+            <wheel_separation>0.49</wheel_separation>
             <wheel_radius>0.08</wheel_radius>
             <!-- 话题配置 -->

Commit message: 新增scan planner规划器，fastlio2回环优化与地图重定位

File: src/scout_description/urdf/chassis.xacro (robot description, xacro)
@@ -70,5 +70,5 @@
     <xacro:wheel_link prefix="front_right"/>
     <xacro:wheel_link prefix="rear_right"/>
-     <link name="mid360_link">
+     <link name="lidar_link">
         <inertial>
             <origin
@@ -117,5 +117,5 @@
     <!-- =================================================================== -->
     <joint name="laser_link_alias_joint" type="fixed">
-        <parent link="mid360_link"/>
+        <parent link="lidar_link"/>
         <child link="laser_link"/>
         <origin xyz="0 0 0" rpy="0 0 0"/>
@@ -130,8 +130,8 @@
         <origin xyz="0.21837 0 0.21508" rpy="0 0 0" />
         <parent link="base_link" />
-        <child link="mid360_link" />
+        <child link="lidar_link" />
     </joint>
     <joint name="imu_joint" type="fixed">
-        <parent link="mid360_link"/>
+        <parent link="lidar_link"/>
         <child link="imu_link"/>
         <origin xyz="0.0 0.0 0.0" rpy="0 0 0"/>
@@ -205,5 +205,5 @@
         filename="$(find livox_mid360_gz_sim)/urdf/mid360_gz_plugin.xacro"/>
     <xacro:livox_mid360_gz_plugin
-        link_name="mid360_link"
+        link_name="lidar_link"
         node_name="livox_mid360_gz_sim"
         frame_id="laser_link"

File: src/scout_description/urdf/scout_mini.urdf.xacro (robot description, xacro)
@@ -5,5 +5,5 @@
     <xacro:include filename="chassis.xacro" />
     <xacro:include filename="/home/hanks/scout_ws/src/piper_description/urdf/my_robot.urdf.xacro" />
-    <xacro:include filename="exp_in_sim.xacro" />
+    <!-- <xacro:include filename="exp_in_sim.xacro" /> -->
     <joint
         name="piper_base_joint"
